Commit message: 0701

File: models/indy7/indy7.urdf (robot description, URDF)
Before this commit: robot indy7, 8 links, 7 joints
Joints:
- joint joint5: origin xyz=-0.16800000 +0.00000000 +0.06900000 rpy=-1.57079632679 0 1.57079632679 -> xyz=-0.16800000 +0.00000000 +0.06900000  rpy=-1.57079632679 0 1.57079632679
